File: circuit/LEDMatrix.kicad_pcb (KiCad board)
At the start: 2 copper layers, 70 x 55 mm, 42 parts, among them J1 LED_PORT1, J2 CONN_USART1, J3 CONN_SWD, J5 LED_PORT2, J6 PWR_IN, U1 AMS1117-3.3, U2 STM32F103C8Tx, U3 TXS0108EPW, U4 JDY-08, U5 XL1509-5.0E1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

Commit message: 合并
Other:
- board text added: "DESIGNER: Uncle Life"
- board text removed: "DESIGNER: LI WEI"
Changed lines of the file:
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@@
     )
+  )
+  (gr_text "DESIGNER: Uncle Life" (at 6.0452 22.8854) (layer B.Cu)
+    (effects (font (size 1.27 1.27) (thickness 0.25)) (justify left mirror))
   )
   (dimension 45 (width 0.15) (layer Cmts.User)
@@
     (effects (font (size 1 1) (thickness 0.15)) (justify left))
   )
-  (gr_text "DESIGNER: LI WEI" (at 2.54 22.86) (layer B.Cu)
-    (effects (font (size 1.27 1.27) (thickness 0.25)) (justify left mirror))
-  )
   (gr_text - (at -33.782 8.001 90) (layer F.SilkS)
